File: board/MECHWARFARE_BOARD.sch (EAGLE design)
At the start: 8 parts, among them J2 5267-3, Q2 FDD4141TO252

Commit message: Moved GND plane to bottom
Moved the ground plane on the board from top to bottom and added heat sink for transistor.
Connections:
- net TURRET_IO renamed N$21
Changed lines of the file:
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@@
 </segment>
 </net>
-<net name="TURRET_IO" class="0">
+<net name="N$21" class="0">
 <segment>
 <pinref part="R1" gate="G$1" pin="1"/>
 <wire x1="137.16" y1="88.9" x2="144.78" y2="88.9" width="0.1524" layer="91"/>
 <pinref part="MS2" gate="G$1" pin="GPIO5"/>
-<label x="142.24" y="93.98" size="1.778" layer="95"/>
 </segment>
 </net>
